Commit message: Many changes
Made ground control interface with the drones through a command message. All commands now go through the same service.

Added a follow mode for the drones.

File: urdf/drone_2.urdf (robot description, URDF)
Before this commit: robot drone, 4 links, 3 joints
Links:
- removed link body
- removed link camera
- removed link camera_link_optical
- removed link hokuyo_link
- added link body_2, mass 0.3; collision box size=0.5 0.5 0.5; visual box size=0.5 0.5 0.5
- added link camera_2, mass 1e-5; collision box size=0.2 0.2 0.2; visual box size=0.2 0.2 0.2
- added link camera_link_optical_2
- added link hokuyo_link_2, mass 1e-5; collision box size=0.1 0.1 0.1; visual box size=0.1 0.1 0.1
Joints:
- removed joint camera_joint
- removed joint camera_optical_joint
- removed joint hokuyo_joint
- added joint camera_joint_2: type fixed, parent body_2, child camera_2, origin xyz=0.25 0 0.25 rpy=0 0 0, axis 0 1 0
- added joint camera_optical_joint_2: type fixed, parent camera_2, child camera_link_optical_2, origin xyz=0 0 0 rpy=-1.5707963267948966 0 -1.5707963267948966
- added joint hokuyo_joint_2: type fixed, parent body_2, child hokuyo_link_2, origin xyz=0 0 -0.05 rpy=0 0 0, axis 0 1 0
